Commit message: Adds differential_drive_controller to the robot

File: src/irobot_description/urdf/irobot.xacro (robot description, xacro)
@@ -70,22 +70,22 @@
 		<!--origin xyz="0.1 0.13 0.1" rpy="0 1.5707 1.5707"/-->
 		<collision name="left_wheel_collision">
-		<origin xyz="0 0 0" rpy="0 1.5707 1.5707"/>
-		<geometry>
-			<cylinder radius="0.1" length="0.05"/>
-		</geometry>
+            <origin xyz="0 0 0" rpy="0 1.5707 1.5707"/>
+            <geometry>
+                <cylinder radius="0.1" length="0.05"/>
+            </geometry>
 		</collision>
 		<visual name="left_wheel_visual">
-		<origin xyz="0 0 0" rpy="0 1.5707 1.5707"/>
-		<geometry>
-			<cylinder radius="0.1" length="0.05"/>
-		</geometry>
+            <origin xyz="0 0 0" rpy="0 1.5707 1.5707"/>
+            <geometry>
+                <cylinder radius="0.1" length="0.05"/>
+            </geometry>
 		</visual>
 		<inertial>
-		<origin xyz="0 0 0" rpy="0 1.5707 1.5707"/>
-		<mass value="5"/>
-		<inertia
-			ixx=".1" ixy="0.0" ixz="0.0"
-			iyy=".1" iyz="0.0"
-			izz=".1"/>
+            <origin xyz="0 0 0" rpy="0 1.5707 1.5707"/>
+            <mass value="5"/>
+            <inertia
+                ixx=".1" ixy="0.0" ixz="0.0"
+                iyy=".1" iyz="0.0"
+                izz=".1"/>
 		</inertial>
 	</link>
@@ -93,26 +93,26 @@
 		<!--origin xyz="0.1 -0.13 0.1" rpy="0 1.5707 1.5707"/-->
 		<collision name="right_wheel_collision">
-		<origin xyz="0 0 0" rpy="0 1.5707 1.5707"/>
-		<geometry>
-			<cylinder radius="0.1" length="0.05"/>
-		</geometry>
+            <origin xyz="0 0 0" rpy="0 1.5707 1.5707"/>
+            <geometry>
+                <cylinder radius="0.1" length="0.05"/>
+            </geometry>
 		</collision>
 		<visual name="right_wheel_visual">
-		<origin xyz="0 0 0" rpy="0 1.5707 1.5707"/>
-		<geometry>
-			<cylinder radius="0.1" length="0.05"/>
-		</geometry>
+            <origin xyz="0 0 0" rpy="0 1.5707 1.5707"/>
+            <geometry>
+                <cylinder radius="0.1" length="0.05"/>
+            </geometry>
 		</visual>
 		<inertial>
-		<origin xyz="0 0 0" rpy="0 1.5707 1.5707"/>
-		<mass value="5"/>
-		<inertia
-			ixx=".1" ixy="0.0" ixz="0.0"
-			iyy=".1" iyz="0.0"
-			izz=".1"/>
+            <origin xyz="0 0 0" rpy="0 1.5707 1.5707"/>
+            <mass value="5"/>
+            <inertia
+                ixx=".1" ixy="0.0" ixz="0.0"
+                iyy=".1" iyz="0.0"
+                izz=".1"/>
 		</inertial>
 	</link>
 	<joint type="continuous" name="left_wheel_hinge">
-		<origin xyz="0 0.275 0" rpy="0 0 0"/>
+		<origin xyz="0 0.28 0" rpy="0 0 0"/>
 		<!--origin xyz="0.1 0.13 0" rpy="0 1.5707 1.5707"/-->
 		<child link="left_wheel"/>
@@ -123,5 +123,5 @@
 	</joint>
 	<joint type="continuous" name="right_wheel_hinge">
-		<origin xyz="0 -0.275 0" rpy="0 0 0"/>
+		<origin xyz="0 -0.28 0" rpy="0 0 0"/>
 		<!--origin xyz="0.1 -0.13 0" rpy="0 1.5707 1.5707"/-->
 		<child link="right_wheel"/>

Commit message: Modifies robot model for smooth movement

File: src/irobot_description/urdf/irobot.xacro (robot description, xacro)
@@ -7,7 +7,7 @@
         <pose> 0 0 0.1 0 0 0 </pose>
         <inertial>
-            <mass value="15.0"/>
-            <origin xyz="0.0 0.0 0.1" rpy="0.0 0.0 0.0"/>
-            <inertia ixx="0.1" ixy="0.0" ixz="0.0" iyy="0.1" iyz="0.0" izz="0.1"/>
+            <mass value="10.0"/>
+            <origin xyz="0 0 0.1" rpy="0 0 0"/>
+            <inertia ixx="0.1" ixy="0" ixz="0" iyy="0.1" iyz="0" izz="0.1"/>
         </inertial>
         <collision name="chassis_collision">
@@ -17,5 +17,5 @@
         </collision>
         <visual name="chassis_visual">
-            <origin xyz="0.0 0.0 0.0" rpy="0.0 0.0 0.0"/>
+            <origin xyz="0 0 0" rpy="0 0 0"/>
             <geometry>
                 <cylinder radius="0.25" length="0.1"/>
@@ -23,5 +23,5 @@
         </visual>
         <collision name='caster_back_collision'>
-            <origin xyz="-0.15 0 -0.05" rpy=" 0 0 0"/>
+            <origin xyz="-0.15 0 -0.0499" rpy=" 0 0 0"/>
             <geometry>
                 <sphere radius="0.05"/>
@@ -39,5 +39,5 @@
 		</collision>
 		<visual name='caster_back_visual'>
-            <origin xyz="-0.15 0 -0.05" rpy=" 0 0 0"/>
+            <origin xyz="-0.15 0 -0.0499" rpy=" 0 0 0"/>
             <geometry>
                 <sphere radius="0.05"/>
@@ -45,5 +45,5 @@
 		</visual>
 		<collision name='caster_front_collision'>
-            <origin xyz="0.15 0 -0.05" rpy=" 0 0 0"/>
+            <origin xyz="0.15 0 -0.0499" rpy=" 0 0 0"/>
             <geometry>
                 <sphere radius="0.05"/>
@@ -61,5 +61,5 @@
 		</collision>
 		<visual name='caster_front_visual'>
-		<origin xyz="0.15 0 -0.05" rpy=" 0 0 0"/>
+		<origin xyz="0.15 0 -0.0499" rpy=" 0 0 0"/>
 		<geometry>
 			<sphere radius="0.05"/>
@@ -85,6 +85,6 @@
             <mass value="5"/>
             <inertia
-                ixx=".1" ixy="0.0" ixz="0.0"
-                iyy=".1" iyz="0.0"
+                ixx=".1" ixy="0" ixz="0"
+                iyy=".1" iyz="0"
                 izz=".1"/>
 		</inertial>
@@ -108,11 +108,11 @@
             <mass value="5"/>
             <inertia
-                ixx=".1" ixy="0.0" ixz="0.0"
-                iyy=".1" iyz="0.0"
+                ixx=".1" ixy="0" ixz="0"
+                iyy=".1" iyz="0"
                 izz=".1"/>
 		</inertial>
 	</link>
 	<joint type="continuous" name="left_wheel_hinge">
-		<origin xyz="0 0.28 0" rpy="0 0 0"/>
+		<origin xyz="0 0.3 0" rpy="0 0 0"/>
 		<!--origin xyz="0.1 0.13 0" rpy="0 1.5707 1.5707"/-->
 		<child link="left_wheel"/>
@@ -123,5 +123,5 @@
 	</joint>
 	<joint type="continuous" name="right_wheel_hinge">
-		<origin xyz="0 -0.28 0" rpy="0 0 0"/>
+		<origin xyz="0 -0.3 0" rpy="0 0 0"/>
 		<!--origin xyz="0.1 -0.13 0" rpy="0 1.5707 1.5707"/-->
 		<child link="right_wheel"/>
